File: design_files/AST1036.sch (EAGLE design)
At the start: 7 parts, among them J1 SM05B, U1 BME680

Commit message: updated documentation
Parts:
- C1: value 10uF -> 1uF; device tinycircuits:AS-ITM-00002 -> tinycircuits:AS-ITM-00410; PARTNO (none) -> AS-ITM-00410; VALUE (none) -> 1uF
- J1: device tinycircuits:AS-ITM-00340 -> tinycircuits:AS-ITM-00340EDGE
Other:
- note added: "Hand Populated: -"
- note added: "Hand Soldered: -"
- note added: "Non Populated: R2"
- note added: "Notes: -"
- note added: "Variant: Standard - R"
- note added: "Wireling Pressure VOC"
- note removed: "NOTES:"
- note removed: "Pres, Hum, VOC Sensor"
